File: disk.sch (EAGLE design)
At the start: 0 parts

Commit message: reworked boards and gerber files
Parts:
- added J1: 1X2-3.5MM, adafruit:1X2-3.5MM
- added LED1: (no value), adafruit:LEDCHIPLED_0805
- added R1: (no value), adafruit:R-US_M0805
Connections:
- new net GND: J1.2, LED1.C
- new net N$1: J1.1, R1.2
- new net N$2: LED1.A, R1.1
Changed lines of the file:
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@@
 </classes>
 <parts>
+<part name="J1" library="adafruit" library_urn="urn:adsk.eagle:library:420" deviceset="1X2" device="-3.5MM" package3d_urn="urn:adsk.eagle:package:6240635/1"/>
+<part name="R1" library="adafruit" library_urn="urn:adsk.eagle:library:420" deviceset="R-US_" device="M0805" package3d_urn="urn:adsk.eagle:package:6240587/1"/>
+<part name="LED1" library="adafruit" library_urn="urn:adsk.eagle:library:420" deviceset="LED" device="CHIPLED_0805" package3d_urn="urn:adsk.eagle:package:6240559/1"/>
+<part name="GND1" library="supply1" library_urn="urn:adsk.eagle:library:371" deviceset="GND" device=""/>
+<part name="GND2" library="supply1" library_urn="urn:adsk.eagle:library:371" deviceset="GND" device=""/>
 </parts>
 <sheets>
@@
 </plain>
 <instances>
+<instance part="J1" gate="G$1" x="104.14" y="50.8" smashed="yes"/>
+<instance part="R1" gate="G$1" x="91.44" y="53.34" smashed="yes">
+<attribute name="NAME" x="87.63" y="54.8386" size="1.778" layer="95"/>
+<attribute name="VALUE" x="87.63" y="50.038" size="1.778" layer="96"/>
+</instance>
+<instance part="LED1" gate="G$1" x="81.28" y="53.34" smashed="yes" rot="R270">
+<attribute name="NAME" x="76.708" y="49.784" size="1.778" layer="95"/>
+<attribute name="VALUE" x="76.708" y="47.625" size="1.778" layer="96"/>
+</instance>
+<instance part="GND1" gate="1" x="73.66" y="45.72" smashed="yes">
+<attribute name="VALUE" x="71.12" y="43.18" size="1.778" layer="96"/>
+</instance>
+<instance part="GND2" gate="1" x="96.52" y="45.72" smashed="yes">
+<attribute name="VALUE" x="93.98" y="43.18" size="1.778" layer="96"/>
+</instance>
 </instances>
 <busses>
 </busses>
 <nets>
+<net name="N$1" class="0">
+<segment>
+<pinref part="J1" gate="G$1" pin="1"/>
+<pinref part="R1" gate="G$1" pin="2"/>
+<wire x1="99.06" y1="53.34" x2="96.52" y2="53.34" width="0.1524" layer="91"/>
+</segment>
+</net>
+<net name="N$2" class="0">
+<segment>
+<pinref part="R1" gate="G$1" pin="1"/>
+<pinref part="LED1" gate="G$1" pin="A"/>
+<wire x1="86.36" y1="53.34" x2="83.82" y2="53.34" width="0.1524" layer="91"/>
+</segment>
+</net>
+<net name="GND" class="0">
+<segment>
+<pinref part="LED1" gate="G$1" pin="C"/>
+<pinref part="GND1" gate="1" pin="GND"/>
+<wire x1="76.2" y1="53.34" x2="73.66" y2="53.34" width="0.1524" layer="91"/>
+<wire x1="73.66" y1="53.34" x2="73.66" y2="48.26" width="0.1524" layer="91"/>
+</segment>
+<segment>
+<pinref part="GND2" gate="1" pin="GND"/>
+<wire x1="96.52" y1="48.26" x2="96.52" y2="50.8" width="0.1524" layer="91"/>
+<pinref part="J1" gate="G$1" pin="2"/>
+<wire x1="96.52" y1="50.8" x2="99.06" y2="50.8" width="0.1524" layer="91"/>
+</segment>
+</net>
 </nets>
 </sheet>
@@
 </schematic>
 </drawing>
+<compatibility>
+<note version="8.2" severity="warning">
+Since Version 8.2, EAGLE supports online libraries. The ids
+of those online libraries will not be understood (or retained)
+with this version.
+</note>
+<note version="8.3" severity="warning">
+Since Version 8.3, EAGLE supports URNs for individual library
+assets (packages, symbols, and devices). The URNs of those assets
+will not be understood (or retained) with this version.
+</note>
+<note version="8.3" severity="warning">
+Since Version 8.3, EAGLE supports the association of 3D packages
+with devices in libraries, schematics, and board files. Those 3D
+packages will not be understood (or retained) with this version.
+</note>
+</compatibility>
 </eagle>
